Commit message: low inertia hover train

File: assets/5_in_drone/urdf/5_in_drone.urdf (robot description, URDF)
Before this commit: robot 5_in_drone, 5 links, 4 joints
Links:
- link body: mass 0.5 -> 0.078
- link prop1: mass None -> 0.001
- link prop2: mass None -> 0.001
- link prop3: mass None -> 0.001
- link prop4: mass None -> 0.001

Commit message: new drone inertia with sysID

File: assets/5_in_drone/urdf/5_in_drone.urdf (robot description, URDF)
Before this commit: robot 5_in_drone, 5 links, 4 joints
Links:
- link body: mass 0.078 -> 0.084
